Commit message: feasible random spawn in gazebo; solve 'static movable object' & 'gravity off' issue

File: urdf/obstacle_1.urdf.xacro (robot description, xacro)
@@ -1,10 +1,11 @@
 <?xml version="1.0"?>
-<robot name="obstacle_2" xmlns:xacro="http://www.ros.org/wiki/xacro">
+<robot name="obstacle_1" xmlns:xacro="http://www.ros.org/wiki/xacro">
 	<xacro:property name="pi" value="3.1415926535897931"/>
 	<gazebo>
 		<static>true</static>
+		<turnGravityOff>false</turnGravityOff>
 	</gazebo>
 	<!-- <link name="world" />-->
-	<link name="base_link">
+	<link name="base_link_1">
 		<inertial>
 			<origin xyz="0 0 0" rpy="0 0 0"/>

File: urdf/obstacle_3.urdf.xacro (robot description, xacro)
@@ -1,10 +1,11 @@
 <?xml version="1.0"?>
-<robot name="obstacle_1" xmlns:xacro="http://www.ros.org/wiki/xacro">
+<robot name="obstacle_3" xmlns:xacro="http://www.ros.org/wiki/xacro">
 	<xacro:property name="pi" value="3.1415926535897931"/>
 	<gazebo>
 		<static>true</static>
+		<turnGravityOff>false</turnGravityOff>
 	</gazebo>
 	<!-- <link name="world" />-->
-	<link name="base_link">
+	<link name="base_link_3">
 		<inertial>
 			<origin xyz="0 0 0" rpy="0 0 0"/>

Commit message: set start and goal area as independent object in gazebo & still exist an issue about distance checking

File: urdf/obstacle_1.urdf.xacro (robot description, xacro)
@@ -16,5 +16,5 @@
 			<origin xyz="0 0 0" rpy="0 0 0"/>
 			<geometry>
-				<box size="1 1 1" />
+				<box size="1.2 10 1.2" />
 			</geometry>
 		</collision>
@@ -22,5 +22,5 @@
 			<origin xyz="0 0 0" rpy="0 0 0"/>
 			<geometry>
-				<box size="1 1 1" />
+				<box size="1.2 10 1.2" />
 			</geometry>
 		</visual>

File: urdf/obstacle_2.urdf.xacro (robot description, xacro)
@@ -16,5 +16,5 @@
 			<origin xyz="0 0 0" rpy="0 0 0"/>
 			<geometry>
-				<box size="1 1 1" />
+				<box size="1.2 10 1.2" />
 			</geometry>
 		</collision>
@@ -22,5 +22,5 @@
 			<origin xyz="0 0 0" rpy="0 0 0"/>
 			<geometry>
-				<box size="1 1 1" />
+				<box size="1.2 10 1.2" />
 			</geometry>
 		</visual>

File: urdf/obstacle_3.urdf.xacro (robot description, xacro)
@@ -16,5 +16,5 @@
 			<origin xyz="0 0 0" rpy="0 0 0"/>
 			<geometry>
-				<box size="1 1 1" />
+				<box size="1.2 10 1.2" />
 			</geometry>
 		</collision>
@@ -22,5 +22,5 @@
 			<origin xyz="0 0 0" rpy="0 0 0"/>
 			<geometry>
-				<box size="1 1 1" />
+				<box size="1.2 10 1.2" />
 			</geometry>
 		</visual>
